File: power-misc.sch (KiCad schematic (older format))
At the start: 4 parts, among them U1 STM32F411-LQFP64, U2 STM32F411-LQFP64

Commit message: Did some stuff
Parts:
- gave numbers to parts that had none: 2
Changed lines of the file:
@@
 $EndComp
 $Comp
-L R R?
+L R R1
 U 1 1 56AE4DF0
 P 3400 3550
-F 0 "R?" V 3480 3550 50  0000 C CNN
+F 0 "R1" V 3480 3550 50  0000 C CNN
 F 1 "100K" V 3400 3550 50  0000 C CNN
 F 2 "" V 3330 3550 30  0000 C CNN
@@
 $EndComp
 $Comp
-L R R?
+L R R2
 U 1 1 56AE4DF7
 P 5250 3550
-F 0 "R?" V 5330 3550 50  0000 C CNN
+F 0 "R2" V 5330 3550 50  0000 C CNN
 F 1 "100K" V 5250 3550 50  0000 C CNN
 F 2 "" V 5180 3550 30  0000 C CNN
@@
 $EndComp
 $Comp
-L +3.3V #PWR?
+L +3.3V #PWR7
 U 1 1 56AE4DFE
 P 3600 3500
-F 0 "#PWR?" H 3600 3350 50  0001 C CNN
+F 0 "#PWR7" H 3600 3350 50  0001 C CNN
 F 1 "+3.3V" H 3600 3640 50  0000 C CNN
 F 2 "" H 3600 3500 60  0000 C CNN
@@
 $EndComp
 $Comp
-L GND #PWR?
+L GND #PWR8
 U 1 1 56AE4E04
 P 5450 3600
-F 0 "#PWR?" H 5450 3350 50  0001 C CNN
+F 0 "#PWR8" H 5450 3350 50  0001 C CNN
 F 1 "GND" H 5450 3450 50  0000 C CNN
 F 2 "" H 5450 3600 60  0000 C CNN
